File: uameter/uameter.sch (KiCad schematic (older format))
At the start: 7 parts

Commit message: uameter: pcb rev1
Parts:
- added P2: CONN_01X02, Pin_Headers:Pin_Header_Straight_1x02, symbol CONN_01X02
- added P3: CONN_01X04, Pin_Headers:Pin_Header_Straight_1x04, symbol CONN_01X04
- added R2: 10k, Resistors_SMD:R_0603_HandSoldering, symbol R
- added U2: TL081, Housings_SOIC:SOIC-8_3.9x4.9mm_Pitch1.27mm, symbol TL081
- C1, C2: renamed from C?; footprint (none) -> Capacitors_SMD:C_0603_HandSoldering
- P1: renamed from P?; footprint (none) -> Connect:USB_Micro-B
- Q1: renamed from Q?; footprint (none) -> TO_SOT_Packages_SMD:SOT-23
- R1: renamed from R?; footprint (none) -> Resistors_SMD:R_0603_HandSoldering
- R3: renamed from R?; value R -> 0.2R; footprint (none) -> Resistors_SMD:R_0603_HandSoldering
- gave numbers to parts that had none: 1
Connections:
- net +3V3: now also C2.1, Q1.3 (S), P3.1 (P1), U2.3 (+), U2.7 (V+)
- net +5V: now also C1.1
- net GND: now also P1.6 (shield), P2.2 (P2), P3.4 (P4), R2.2, U2.4 (V-)
- net at R1.1, R3.2: now also Q1.1 (D)
- net PMOS_IN: now reaches Q1.2 (G)
- net PMOS_IN: now also P3.2 (P2), R2.1
- net D+: no longer names the net of P1.3 (D+)
- net D-: no longer names the net of P1.2 (D-)
- net VCC renamed V_OUT
- net V_OUT: now also P2.1 (P1), U2.2 (-)
- new net OP_OUT: P3.3 (P3), U2.6
- no-connect marks 0 -> 3
Other:
- moved on the sheet: C1, C2, Q1, R1, R3
